Commit message: Reset head camera depth joint origin

File: src/pincer/assets/xlerobot/xlerobot_front.urdf (robot description, URDF)
Before this commit: robot fetch, 32 links, 31 joints
Joints:
- joint head_camera_depth_joint: origin xyz=0 0.045 0 rpy=0 0 0 -> xyz=0 0 0 rpy=0 0 0

Commit message: Adjust head camera and depth frame offsets

File: src/pincer/assets/xlerobot/xlerobot_front.urdf (robot description, URDF)
Before this commit: robot fetch, 32 links, 31 joints
Joints:
- joint head_camera_depth_joint: origin xyz=0 0 0 rpy=0 0 0 -> xyz=0 0.045 0 rpy=0 0 0
- joint head_camera_joint: origin xyz=0.055 0 0.0225 rpy=0 0 0 -> xyz=0.035 0 0.04 rpy=0 0 0

Commit message: Adjust head camera pose and use color intrinsics
Move head camera forward and slightly lower in URDF (xyz updated).
When align_to_color is true, use the color stream intrinsics;
otherwise fall back to depth intrinsics.

File: src/pincer/assets/xlerobot/xlerobot_front.urdf (robot description, URDF)
Before this commit: robot fetch, 32 links, 31 joints
Joints:
- joint head_camera_joint: origin xyz=0.035 0 0.04 rpy=0 0 0 -> xyz=0.055 0 0.0225 rpy=0 0 0
